Commit message: fixed xmlns in urdf xacro files. fixed cmd vel for simulated gvrbot

File: models/robots/basic_colors.urdf.xacro (robot description, xacro)
@@ -1,43 +1,43 @@
 <?xml version="1.0"?>
-<robot>
-  <macro name="Black">
+<robot xmlns:xacro="http://www.ros.org/wiki/xacro">
+  <xacro:macro name="Black">
     <material name="black">
       <color rgba="0.0 0.0 0.0 1.0"/>
     </material>
-  </macro>
-  <macro name="Blue">
+  </xacro:macro>
+  <xacro:macro name="Blue">
     <material name="blue">
       <color rgba="0.0 0.0 0.8 1.0"/>
     </material>
-  </macro>
-  <macro name="Green">
+  </xacro:macro>
+  <xacro:macro name="Green">
     <material name="green">
       <color rgba="0.0 0.8 0.0 1.0"/>
     </material>
-  </macro>
-  <macro name="Gray">
+  </xacro:macro>
+  <xacro:macro name="Gray">
     <material name="gray">
       <color rgba="0.7 0.7 0.7 1.0"/>
     </material>
-  </macro>
-  <macro name="DarkGray">
+  </xacro:macro>
+  <xacro:macro name="DarkGray">
     <material name="darkGray">
       <color rgba="0.3 0.3 0.3 1.0"/>
     </material>
-  </macro>
-  <macro name="Red">
+  </xacro:macro>
+  <xacro:macro name="Red">
     <material name="red">
       <color rgba="0.8 0.0 0.0 1.0"/>
     </material>
-  </macro>
-  <macro name="White">
+  </xacro:macro>
+  <xacro:macro name="White">
     <material name="white">
       <color rgba="1.0 1.0 1.0 1.0"/>
     </material>
-  </macro>
-  <macro name="Yellow">
+  </xacro:macro>
+  <xacro:macro name="Yellow">
     <material name="yellow">
       <color rgba="0.8 0.8 0.0 1.0"/>
     </material>
-  </macro>
+  </xacro:macro>
 </robot>

File: models/robots/frame_8020.urdf.xacro (robot description, xacro)
@@ -1,5 +1,5 @@
-<robot xmlns:xacro="http://playerstage.sourceforge.net/gazebo/xmlschema/#interface">
-    <property name="M_PI" value="3.14159"/>
-    <macro name="frame_8020" params="parent offset_x offset_y offset_z">
+<robot xmlns:xacro="http://www.ros.org/wiki/xacro">
+    <xacro:property name="M_PI" value="3.14159"/>
+    <xacro:macro name="frame_8020" params="parent offset_x offset_y offset_z">
         <joint name="frame_8020_joint" type="fixed">
             <origin xyz="${offset_x} ${offset_y} ${offset_z}" rpy="0 0 ${-M_PI/2}" />
@@ -31,4 +31,4 @@
             </collision>
         </link>
-   </macro>
+   </xacro:macro>
 </robot>

File: models/robots/gvrbot.urdf.xacro (robot description, xacro)
@@ -1,15 +1,12 @@
 <?xml version="1.0"?>
-<robot name="gvrbot"
-    xmlns:sensor="http://playerstage.sourceforge.net/gazebo/xmlschema/#sensor"
-    xmlns:controller="http://playerstage.sourceforge.net/gazebo/xmlschema/#controller"
-    xmlns:interface="http://playerstage.sourceforge.net/gazebo/xmlschema/#interface">
+<robot name="gvrbot" xmlns:xacro="http://www.ros.org/wiki/xacro">
     <!-- Included URDF Files    -->
-    <include filename="$(find gvrbot)/models/robots/gvrbot_base.urdf.xacro" />
+    <xacro:include filename="$(find gvrbot)/models/robots/gvrbot_base.urdf.xacro" />
     <gvr_base_macro />
-    <include filename="$(find gvrbot)/models/robots/frame_8020.urdf.xacro" />
+    <xacro:include filename="$(find gvrbot)/models/robots/frame_8020.urdf.xacro" />
     <frame_8020 parent="base_link" offset_x="0.28" offset_y="0.135" offset_z="-0.115"/>
-   <arg name="gpu" default="false"/>
-  <property name="gpu" value="$(arg gpu)" />
-  <include filename="$(find velodyne_description)/urdf/HDL-32E.urdf.xacro"/>
+   <xacro:arg name="gpu" default="false"/>
+  <xacro:property name="gpu" value="$(arg gpu)" />
+  <xacro:include filename="$(find velodyne_description)/urdf/HDL-32E.urdf.xacro"/>
   <HDL-32E parent="base_link" name="velodyne2" topic="/velodyne_points2" hz="10" samples="220" gpu="${gpu}">
     <origin xyz="-0.028 -0.006 0.46" rpy="0 0 0" />

File: models/robots/gvrbot_base.urdf.xacro (robot description, xacro)
@@ -1,8 +1,6 @@
 <?xml version="1.0"?>
 <robot
-    xmlns:xacro="http://playerstage.sourceforge.net/gazebo/xmlschema/#interface"
-    xmlns:sensor="http://playerstage.sourceforge.net/gazebo/xmlschema/#sensor"
-    xmlns:controller="http://playerstage.sourceforge.net/gazebo/xmlschema/#controller"
-    xmlns:interface="http://playerstage.sourceforge.net/gazebo/xmlschema/#interface">
+    xmlns:xacro="http://www.ros.org/wiki/xacro"
+    xmlns:interface="http://www.ros.org/wiki/xacro/#interface">
     <xacro:include filename="$(find gvrbot)/models/robots/inertial_tensors.urdf.xacro" />
     <xacro:include filename="$(find gvrbot)/models/robots/single_wheel.urdf.xacro" />
@@ -10,17 +8,17 @@
     <xacro:include filename="$(find gvrbot)/models/robots/plexiglass_mount.urdf.xacro" />
     <!-- Properties (Constants) -->
-    <property name="M_PI" value="3.14159"/>
-    <property name="base_size_x" value="0.380" />
-    <property name="base_size_y" value="0.3" />
-    <property name="base_size_z" value="0.085" />
-    <property name="base_mass" value="25.0" />
-    <property name="wheel_radius_big" value="0.085" />
-    <property name="wheel_size_y" value="0.0825" />
-    <property name="wheel_mass" value="0.1" />
-    <property name="wheel_offset_z_from_base_link" value="-${wheel_radius_big}" />
+    <xacro:property name="M_PI" value="3.14159"/>
+    <xacro:property name="base_size_x" value="0.380" />
+    <xacro:property name="base_size_y" value="0.3" />
+    <xacro:property name="base_size_z" value="0.085" />
+    <xacro:property name="base_mass" value="25.0" />
+    <xacro:property name="wheel_radius_big" value="0.085" />
+    <xacro:property name="wheel_size_y" value="0.0825" />
+    <xacro:property name="wheel_mass" value="0.1" />
+    <xacro:property name="wheel_offset_z_from_base_link" value="-${wheel_radius_big}" />
       <material name="army_green">
     <color rgba="${42/255} ${46/255} ${18/255} 1.0"/>
   </material>
-    <macro name="gvr_base_macro">
+    <xacro:macro name="gvr_base_macro">
         <!-- Links and Joints (i.e., the robot) -->
         <link name="base_footprint"/>
@@ -83,8 +81,9 @@
                 <robotNamespace>/</robotNamespace>
                 <robotBaseFrame>base_link</robotBaseFrame>
-                <commandTopic>/gvrbot/cmd_vel</commandTopic>
+                <commandTopic>/cmd_vel</commandTopic>
                 <publishOdometryTf>1</publishOdometryTf>
                 <publishOdometryMsg>1</publishOdometryMsg>
                 <odometryTopic>/gvrbot/odom</odometryTopic>
+                <odometryFrame>odom</odometryFrame>
         </plugin>
         <plugin name="p3d_base_controller" filename="libgazebo_ros_p3d.so">
@@ -109,6 +108,8 @@
           <headingDrift>0.0</headingDrift>
           <headingGaussianNoise>0.05</headingGaussianNoise>
+          <xyzOffset>0 0 0</xyzOffset>
+          <rpyOffset>0 0 0</rpyOffset>
         </plugin>
         </gazebo>
-    </macro>
+    </xacro:macro>
 </robot>

File: models/robots/gvrbot_velodyne.urdf.xacro (robot description, xacro)
@@ -1,11 +1,8 @@
 <?xml version="1.0"?>
-<robot name="gvrbot"
-    xmlns:sensor="http://playerstage.sourceforge.net/gazebo/xmlschema/#sensor"
-    xmlns:controller="http://playerstage.sourceforge.net/gazebo/xmlschema/#controller"
-    xmlns:interface="http://playerstage.sourceforge.net/gazebo/xmlschema/#interface">
+<robot name="gvrbot" xmlns:xacro="http://www.ros.org/wiki/xacro">
     <!-- Included URDF Files -->
-    <include filename="$(find gvrbot)/models/robots/gvr_base.urdf.xacro" />
-    <include filename="$(find usma_velodyne)/urdf/velodyne.urdf.xacro" />
-  <!--  <include filename="$(find pointgrey_camera_description)/urdf/pointgrey_flea3.urdf.xacro" /> -->
+    <xacro:include filename="$(find gvrbot)/models/robots/gvr_base.urdf.xacro" />
+    <xacro:include filename="$(find usma_velodyne)/urdf/velodyne.urdf.xacro" />
+  <!--  <xacro:include filename="$(find pointgrey_camera_description)/urdf/pointgrey_flea3.urdf.xacro" /> -->
     <gvr_base_macro />
     <plexiglass_mount_macro />

File: models/robots/inertial_tensors.urdf.xacro (robot description, xacro)
@@ -1,14 +1,14 @@
 <?xml version="1.0"?>
-<robot>
-  <macro name="rectangular_prism_tensor" params="mass len_x len_y len_z">
+<robot xmlns:xacro="http://www.ros.org/wiki/xacro">
+  <xacro:macro name="rectangular_prism_tensor" params="mass len_x len_y len_z">
     <inertia   ixx="${ mass / 3 * ( len_y * len_y + len_z * len_z ) }" ixy="${ mass / 4 * len_x * len_y }" ixz="${ mass / 4 * len_x * len_z }"
                iyy="${ mass / 3 * ( len_y * len_y + len_z * len_z ) }" iyz="${ mass / 4 * len_y * len_z }"
                izz="${ mass / 3 * ( len_y * len_y + len_z * len_z ) }" />
-  </macro>
+  </xacro:macro>
   <!-- Z axis through the center of top and bottom  -->
-  <macro name="cylinder_tensor" params="mass radius height">
+  <xacro:macro name="cylinder_tensor" params="mass radius height">
     <inertia   ixx="${ mass / 12 * height * height + mass / 4 * radius * radius }" ixy="0.0" ixz="0.0"
                iyy="${ mass / 12 * height * height + mass / 4 * radius * radius }" iyz="0.0"
                izz="${ mass / 2 * radius * radius }" />
-  </macro>
+  </xacro:macro>
 </robot>

File: models/robots/plexiglass_mount.urdf.xacro (robot description, xacro)
@@ -1,8 +1,4 @@
 <?xml version="1.0"?>
-<robot
-  xmlns:sensor="http://playerstage.sourceforge.net/gazebo/xmlschema/#sensor"
-  xmlns:controller="http://playerstage.sourceforge.net/gazebo/xmlschema/#controller"
-  xmlns:interface="http://playerstage.sourceforge.net/gazebo/xmlschema/#interface"
-  xmlns:xacro="http://playerstage.sourceforge.net/gazebo/xmlschema/#interface">
+<robot xmlns:xacro="http://www.ros.org/wiki/xacro">
  <xacro:include filename="$(find gvrbot)/models/robots/basic_colors.urdf.xacro" />
  <xacro:include filename="$(find gvrbot)/models/robots/inertial_tensors.urdf.xacro" />

File: models/robots/single_wheel.urdf.xacro (robot description, xacro)
@@ -1,8 +1,5 @@
 <?xml version="1.0"?>
 <robot
-  xmlns:sensor="http://playerstage.sourceforge.net/gazebo/xmlschema/#sensor"
-  xmlns:controller="http://playerstage.sourceforge.net/gazebo/xmlschema/#controller"
-  xmlns:interface="http://playerstage.sourceforge.net/gazebo/xmlschema/#interface"
-  xmlns:xacro="http://playerstage.sourceforge.net/gazebo/xmlschema/#interface">
+  xmlns:xacro="http://www.ros.org/wiki/xacro">
  <xacro:include filename="$(find gvrbot)/models/robots/basic_colors.urdf.xacro" />
  <xacro:include filename="$(find gvrbot)/models/robots/inertial_tensors.urdf.xacro" />
