Commit message: Adjusting the gvrbot model and working on gazebo sim launch

File: models/robots/gvrbot_base.urdf.xacro (robot description, xacro)
@@ -5,8 +5,8 @@
     xmlns:controller="http://playerstage.sourceforge.net/gazebo/xmlschema/#controller"
     xmlns:interface="http://playerstage.sourceforge.net/gazebo/xmlschema/#interface">
-    <xacro:include filename="$(find gvr_bot)/models/robots/inertial_tensors.urdf.xacro" />
-    <xacro:include filename="$(find gvr_bot)/models/robots/single_wheel.urdf.xacro" />
-    <xacro:include filename="$(find gvr_bot)/models/robots/basic_colors.urdf.xacro" />
-    <xacro:include filename="$(find gvr_bot)/models/robots/plexiglass_mount.urdf.xacro" />
+    <xacro:include filename="$(find gvrbot)/models/robots/inertial_tensors.urdf.xacro" />
+    <xacro:include filename="$(find gvrbot)/models/robots/single_wheel.urdf.xacro" />
+    <xacro:include filename="$(find gvrbot)/models/robots/basic_colors.urdf.xacro" />
+    <xacro:include filename="$(find gvrbot)/models/robots/plexiglass_mount.urdf.xacro" />
     <!-- Properties (Constants) -->
     <property name="M_PI" value="3.14159"/>
@@ -19,4 +19,7 @@
     <property name="wheel_mass" value="0.1" />
     <property name="wheel_offset_z_from_base_link" value="-${wheel_radius_big}" />
+      <material name="army_green">
+    <color rgba="${42/255} ${46/255} ${18/255} 1.0"/>
+  </material>
     <macro name="gvr_base_macro">
         <!-- Links and Joints (i.e., the robot) -->
@@ -37,7 +40,7 @@
                 <origin xyz="${base_size_x - 0.05} 0.0 -${base_size_z * 2}" rpy="0 0 1.57" />
                 <geometry>
-                    <mesh filename="package://gvr_bot/models/meshes/base_link.STL"/>
+                    <mesh filename="package://gvrbot/models/meshes/gvrbot_base.STL"/>
                 </geometry>
-                <Gray />
+                <material name="army_green"/>
             </visual>
             <!--visual>
@@ -80,8 +83,8 @@
                 <robotNamespace>/</robotNamespace>
                 <robotBaseFrame>base_link</robotBaseFrame>
-                <commandTopic>/gvr_bot/cmd_vel</commandTopic>
+                <commandTopic>/gvrbot/cmd_vel</commandTopic>
                 <publishOdometryTf>1</publishOdometryTf>
                 <publishOdometryMsg>1</publishOdometryMsg>
-                <odometryTopic>/gvr_bot/odom</odometryTopic>
+                <odometryTopic>/gvrbot/odom</odometryTopic>
         </plugin>
         <plugin name="p3d_base_controller" filename="libgazebo_ros_p3d.so">
@@ -89,5 +92,5 @@
           <updateRate>50.0</updateRate>
           <bodyName>base_link</bodyName>
-          <topicName>/gvr_bot/ground_truth/state</topicName>
+          <topicName>/gvrbot/ground_truth/state</topicName>
           <gaussianNoise>0.01</gaussianNoise>
           <frameName>world</frameName>
@@ -99,5 +102,5 @@
           <updateRate>50.0</updateRate>
           <bodyName>base_link</bodyName>
-          <topicName>/gvr_bot/imu_quat</topicName>
+          <topicName>/gvrbot/imu_quat</topicName>
           <accelDrift>0.0 0.0 0.0</accelDrift>
           <accelGaussianNoise>0.1 0.1 0.1</accelGaussianNoise>

File: models/robots/gvrbot_velodyne.urdf.xacro (robot description, xacro)
@@ -1,9 +1,9 @@
 <?xml version="1.0"?>
-<robot name="gvr_bot"
+<robot name="gvrbot"
     xmlns:sensor="http://playerstage.sourceforge.net/gazebo/xmlschema/#sensor"
     xmlns:controller="http://playerstage.sourceforge.net/gazebo/xmlschema/#controller"
     xmlns:interface="http://playerstage.sourceforge.net/gazebo/xmlschema/#interface">
     <!-- Included URDF Files -->
-    <include filename="$(find gvr_bot)/models/robots/gvr_base.urdf.xacro" />
+    <include filename="$(find gvrbot)/models/robots/gvr_base.urdf.xacro" />
     <include filename="$(find usma_velodyne)/urdf/velodyne.urdf.xacro" />
   <!--  <include filename="$(find pointgrey_camera_description)/urdf/pointgrey_flea3.urdf.xacro" /> -->

File: models/robots/plexiglass_mount.urdf.xacro (robot description, xacro)
@@ -5,6 +5,6 @@
   xmlns:interface="http://playerstage.sourceforge.net/gazebo/xmlschema/#interface"
   xmlns:xacro="http://playerstage.sourceforge.net/gazebo/xmlschema/#interface">
- <xacro:include filename="$(find gvr_bot)/models/robots/basic_colors.urdf.xacro" />
- <xacro:include filename="$(find gvr_bot)/models/robots/inertial_tensors.urdf.xacro" />
+ <xacro:include filename="$(find gvrbot)/models/robots/basic_colors.urdf.xacro" />
+ <xacro:include filename="$(find gvrbot)/models/robots/inertial_tensors.urdf.xacro" />
   <!-- Properties (Constants) -->
   <xacro:property name="M_PI" value="3.14159" />
@@ -19,5 +19,5 @@
           <origin xyz="-0.25 -0.125 -0.03" rpy="0 0 0"/>
           <geometry>
-              <mesh filename="package://gvr_bot/models/meshes/mount_link.STL" />
+              <mesh filename="package://gvrbot/models/meshes/mount_link.STL" />
           </geometry>
           <White />

File: models/robots/single_wheel.urdf.xacro (robot description, xacro)
@@ -5,6 +5,6 @@
   xmlns:interface="http://playerstage.sourceforge.net/gazebo/xmlschema/#interface"
   xmlns:xacro="http://playerstage.sourceforge.net/gazebo/xmlschema/#interface">
- <xacro:include filename="$(find gvr_bot)/models/robots/basic_colors.urdf.xacro" />
- <xacro:include filename="$(find gvr_bot)/models/robots/inertial_tensors.urdf.xacro" />
+ <xacro:include filename="$(find gvrbot)/models/robots/basic_colors.urdf.xacro" />
+ <xacro:include filename="$(find gvrbot)/models/robots/inertial_tensors.urdf.xacro" />
   <!-- Properties (Constants) -->
   <xacro:property name="M_PI" value="3.14159" />

Commit message: working on fixing simulated diff drive

File: models/robots/gvrbot_base.urdf.xacro (robot description, xacro)
@@ -5,6 +5,6 @@
     <xacro:include filename="$(find gvrbot)/models/robots/inertial_tensors.urdf.xacro" />
     <xacro:include filename="$(find gvrbot)/models/robots/single_wheel.urdf.xacro" />
+    <xacro:include filename="$(find gvrbot)/models/robots/track_wheel.urdf.xacro" />
     <xacro:include filename="$(find gvrbot)/models/robots/basic_colors.urdf.xacro" />
-    <xacro:include filename="$(find gvrbot)/models/robots/plexiglass_mount.urdf.xacro" />
     <!-- Properties (Constants) -->
     <xacro:property name="M_PI" value="3.14159"/>
@@ -28,5 +28,11 @@
           <child link="base_footprint"/>
         </joint>
-        <link name="base_link">
+        <link name="base_link"/>
+         <joint name="chasis_to_bl" type="fixed">
+          <origin xyz="0.0 0.0 0.0" rpy="0.0 0.0 0.0" />
+          <parent link="base_link"/>
+          <child link="chasis_link"/>
+        </joint>
+        <link name="chasis_link">
             <inertial>
                 <mass value="${base_mass}" />
@@ -56,16 +62,20 @@
             </collision>
         </link>
-        <tracked_wheel parent="base_link" prefix="left_0"  offset_x=" 0.25100" offset_y=" ${base_size_y / 2}" offset_z="${wheel_offset_z_from_base_link}      " reflect="1" radius="${wheel_radius_big}" height="${wheel_size_y}" mass="${wheel_mass}"/>
-        <tracked_wheel parent="base_link" prefix="left_1"  offset_x=" 0.00000" offset_y=" ${base_size_y / 2}" offset_z="${wheel_offset_z_from_base_link-0.005}" reflect="1" radius="${wheel_radius_big}" height="${wheel_size_y}" mass="${wheel_mass}"/>
-        <tracked_wheel parent="base_link" prefix="left_2"  offset_x="-0.25100" offset_y=" ${base_size_y / 2}" offset_z="${wheel_offset_z_from_base_link}      " reflect="1" radius="${wheel_radius_big}" height="${wheel_size_y}" mass="${wheel_mass}"/>
+        <tracked_wheel2 parent="base_link" prefix="left_0"  offset_x=" 0.25100" offset_y=" ${base_size_y / 2}" offset_z="${wheel_offset_z_from_base_link}      " reflect="1" radius="${wheel_radius_big}" height="${wheel_size_y}" mass="${wheel_mass}"/>
+        <tracked_wheel2 parent="base_link" prefix="left_1"  offset_x=" 0.00000" offset_y=" ${base_size_y / 2}" offset_z="${wheel_offset_z_from_base_link-0.005}" reflect="1" radius="${wheel_radius_big}" height="${wheel_size_y}" mass="${wheel_mass}"/>
+        <tracked_wheel2 parent="base_link" prefix="left_2"  offset_x="-0.25100" offset_y=" ${base_size_y / 2}" offset_z="${wheel_offset_z_from_base_link}      " reflect="1" radius="${wheel_radius_big}" height="${wheel_size_y}" mass="${wheel_mass}"/>
+        <tracked_wheel2 parent="base_link" prefix="right_0" offset_x=" 0.25100" offset_y="-${base_size_y / 2}" offset_z="${wheel_offset_z_from_base_link}      " reflect="1" radius="${wheel_radius_big}" height="${wheel_size_y}" mass="${wheel_mass}"/>
+        <tracked_wheel2 parent="base_link" prefix="right_1" offset_x=" 0.00000" offset_y="-${base_size_y / 2}" offset_z="${wheel_offset_z_from_base_link-0.005}" reflect="1" radius="${wheel_radius_big}" height="${wheel_size_y}" mass="${wheel_mass}"/>
+        <tracked_wheel2 parent="base_link" prefix="right_2" offset_x="-0.25100" offset_y="-${base_size_y / 2}" offset_z="${wheel_offset_z_from_base_link}      " reflect="1" radius="${wheel_radius_big}" height="${wheel_size_y}" mass="${wheel_mass}"/>
+        <!--
+        <tracked_wheel parent="base_link" prefix="right_3" offset_x="-0.10550" offset_y="-${base_size_y / 2}" offset_z="${wheel_offset_z_from_base_link}      " reflect="1" radius="${wheel_radius_big}" height="${wheel_size_y}" mass="${wheel_mass}"/>
+        <tracked_wheel parent="base_link" prefix="right_4" offset_x=" 0.10550" offset_y="-${base_size_y / 2}" offset_z="${wheel_offset_z_from_base_link}      " reflect="1" radius="${wheel_radius_big}" height="${wheel_size_y}" mass="${wheel_mass}"/>
+        <tracked_wheel parent="base_link" prefix="right_5" offset_x=" 0.00500" offset_y="-${base_size_y / 2}" offset_z="${wheel_offset_z_from_base_link+0.005}" reflect="1" radius="${wheel_radius_big}" height="${wheel_size_y}" mass="${wheel_mass}"/>
         <tracked_wheel parent="base_link" prefix="left_3"  offset_x=" 0.10550" offset_y=" ${base_size_y / 2}" offset_z="${wheel_offset_z_from_base_link}      " reflect="1" radius="${wheel_radius_big}" height="${wheel_size_y}" mass="${wheel_mass}"/>
         <tracked_wheel parent="base_link" prefix="left_4"  offset_x="-0.10550" offset_y=" ${base_size_y / 2}" offset_z="${wheel_offset_z_from_base_link}      " reflect="1" radius="${wheel_radius_big}" height="${wheel_size_y}" mass="${wheel_mass}"/>
         <tracked_wheel parent="base_link" prefix="left_5"  offset_x=" 0.00500" offset_y=" ${base_size_y / 2}" offset_z="${wheel_offset_z_from_base_link+0.005}" reflect="1" radius="${wheel_radius_big}" height="${wheel_size_y}" mass="${wheel_mass}"/>
-        <tracked_wheel parent="base_link" prefix="right_0" offset_x=" 0.25100" offset_y="-${base_size_y / 2}" offset_z="${wheel_offset_z_from_base_link}      " reflect="1" radius="${wheel_radius_big}" height="${wheel_size_y}" mass="${wheel_mass}"/>
-        <tracked_wheel parent="base_link" prefix="right_1" offset_x=" 0.00000" offset_y="-${base_size_y / 2}" offset_z="${wheel_offset_z_from_base_link-0.005}" reflect="1" radius="${wheel_radius_big}" height="${wheel_size_y}" mass="${wheel_mass}"/>
-        <tracked_wheel parent="base_link" prefix="right_2" offset_x="-0.25100" offset_y="-${base_size_y / 2}" offset_z="${wheel_offset_z_from_base_link}      " reflect="1" radius="${wheel_radius_big}" height="${wheel_size_y}" mass="${wheel_mass}"/>
-        <tracked_wheel parent="base_link" prefix="right_3" offset_x="-0.10550" offset_y="-${base_size_y / 2}" offset_z="${wheel_offset_z_from_base_link}      " reflect="1" radius="${wheel_radius_big}" height="${wheel_size_y}" mass="${wheel_mass}"/>
-        <tracked_wheel parent="base_link" prefix="right_4" offset_x=" 0.10550" offset_y="-${base_size_y / 2}" offset_z="${wheel_offset_z_from_base_link}      " reflect="1" radius="${wheel_radius_big}" height="${wheel_size_y}" mass="${wheel_mass}"/>
-        <tracked_wheel parent="base_link" prefix="right_5" offset_x=" 0.00500" offset_y="-${base_size_y / 2}" offset_z="${wheel_offset_z_from_base_link+0.005}" reflect="1" radius="${wheel_radius_big}" height="${wheel_size_y}" mass="${wheel_mass}"/>
+                <leftJoints>left_0_wheel_joint left_1_wheel_joint left_2_wheel_joint left_3_wheel_joint left_4_wheel_joint left_5_wheel_joint</leftJoints>
+                <rightJoints>right_0_wheel_joint right_1_wheel_joint right_2_wheel_joint right_3_wheel_joint right_4_wheel_joint right_5_wheel_joint</rightJoints>
+         -->
         <gazebo>
         <!-- TODO: make custom plugin for this that doesn't require an imu -->
@@ -73,11 +83,11 @@
                 <alwaysOn>true</alwaysOn>
                 <updateRate>50.0</updateRate>
-                <leftJoints>left_0_wheel_joint left_1_wheel_joint left_2_wheel_joint left_3_wheel_joint left_4_wheel_joint left_5_wheel_joint</leftJoints>
-                <rightJoints>right_0_wheel_joint right_1_wheel_joint right_2_wheel_joint right_3_wheel_joint right_4_wheel_joint right_5_wheel_joint</rightJoints>
+                <leftJoints>left_0_wheel_joint left_1_wheel_joint left_2_wheel_joint</leftJoints>
+                <rightJoints>right_0_wheel_joint right_1_wheel_joint right_2_wheel_joint</rightJoints>
                 <wheelSeparation>${base_size_y}</wheelSeparation>
                 <wheelDiameter>${wheel_radius_big*2}</wheelDiameter>
                 <torque>50000</torque>
                 <interface:position name="position_iface_2"/>
-                <robotNamespace>/</robotNamespace>
+                <robotNamespace>/gvrbot</robotNamespace>
                 <robotBaseFrame>base_link</robotBaseFrame>
                 <commandTopic>/cmd_vel</commandTopic>

File: models/robots/single_wheel.urdf.xacro (robot description, xacro)
@@ -46,5 +46,5 @@
       <transmission name="${prefix}_wheel_trans">
         <type>transmission_interface/SimpleTransmission</type>
-        <joint name="${prefix}_wheel_joint">
+        <joint name="${prefix}_wheelt_joint">
           <hardwareInterface>EffortJointInterface</hardwareInterface>
         </joint>

Commit message: exploring other diff drive solutions

File: models/robots/gvrbot_base.urdf.xacro (robot description, xacro)
@@ -6,4 +6,5 @@
     <xacro:include filename="$(find gvrbot)/models/robots/single_wheel.urdf.xacro" />
     <xacro:include filename="$(find gvrbot)/models/robots/track_wheel.urdf.xacro" />
+    <xacro:include filename="$(find gvrbot)/models/robots/track_wheel3.urdf.xacro" />
     <xacro:include filename="$(find gvrbot)/models/robots/basic_colors.urdf.xacro" />
     <!-- Properties (Constants) -->
@@ -28,11 +29,11 @@
           <child link="base_footprint"/>
         </joint>
-        <link name="base_link"/>
-         <joint name="chasis_to_bl" type="fixed">
-          <origin xyz="0.0 0.0 0.0" rpy="0.0 0.0 0.0" />
-          <parent link="base_link"/>
-          <child link="chasis_link"/>
+        <link name="base_link"></link>
+        <joint name="base_link_joint" type="fixed">
+            <origin xyz="0 0 0" rpy="0 0 0" />
+            <parent link="base_link"/>
+            <child link="chassis_link" />
         </joint>
-        <link name="chasis_link">
+        <link name="chassis_link">
             <inertial>
                 <mass value="${base_mass}" />
@@ -62,10 +63,10 @@
             </collision>
         </link>
-        <tracked_wheel2 parent="base_link" prefix="left_0"  offset_x=" 0.25100" offset_y=" ${base_size_y / 2}" offset_z="${wheel_offset_z_from_base_link}      " reflect="1" radius="${wheel_radius_big}" height="${wheel_size_y}" mass="${wheel_mass}"/>
-        <tracked_wheel2 parent="base_link" prefix="left_1"  offset_x=" 0.00000" offset_y=" ${base_size_y / 2}" offset_z="${wheel_offset_z_from_base_link-0.005}" reflect="1" radius="${wheel_radius_big}" height="${wheel_size_y}" mass="${wheel_mass}"/>
-        <tracked_wheel2 parent="base_link" prefix="left_2"  offset_x="-0.25100" offset_y=" ${base_size_y / 2}" offset_z="${wheel_offset_z_from_base_link}      " reflect="1" radius="${wheel_radius_big}" height="${wheel_size_y}" mass="${wheel_mass}"/>
-        <tracked_wheel2 parent="base_link" prefix="right_0" offset_x=" 0.25100" offset_y="-${base_size_y / 2}" offset_z="${wheel_offset_z_from_base_link}      " reflect="1" radius="${wheel_radius_big}" height="${wheel_size_y}" mass="${wheel_mass}"/>
-        <tracked_wheel2 parent="base_link" prefix="right_1" offset_x=" 0.00000" offset_y="-${base_size_y / 2}" offset_z="${wheel_offset_z_from_base_link-0.005}" reflect="1" radius="${wheel_radius_big}" height="${wheel_size_y}" mass="${wheel_mass}"/>
-        <tracked_wheel2 parent="base_link" prefix="right_2" offset_x="-0.25100" offset_y="-${base_size_y / 2}" offset_z="${wheel_offset_z_from_base_link}      " reflect="1" radius="${wheel_radius_big}" height="${wheel_size_y}" mass="${wheel_mass}"/>
+        <tracked_wheel3 parent="base_link" prefix="left_0"  offset_x=" 0.25100" offset_y=" ${base_size_y / 2}" offset_z="${wheel_offset_z_from_base_link}      " reflect="1" radius="${wheel_radius_big}" height="${wheel_size_y}" mass="${wheel_mass}"/>
+        <tracked_wheel3 parent="base_link" prefix="left_1"  offset_x=" 0.00000" offset_y=" ${base_size_y / 2}" offset_z="${wheel_offset_z_from_base_link-0.005}" reflect="1" radius="${wheel_radius_big}" height="${wheel_size_y}" mass="${wheel_mass}"/>
+        <tracked_wheel3 parent="base_link" prefix="left_2"  offset_x="-0.25100" offset_y=" ${base_size_y / 2}" offset_z="${wheel_offset_z_from_base_link}      " reflect="1" radius="${wheel_radius_big}" height="${wheel_size_y}" mass="${wheel_mass}"/>
+        <tracked_wheel3 parent="base_link" prefix="right_0" offset_x=" 0.25100" offset_y="-${base_size_y / 2}" offset_z="${wheel_offset_z_from_base_link}      " reflect="1" radius="${wheel_radius_big}" height="${wheel_size_y}" mass="${wheel_mass}"/>
+        <tracked_wheel3 parent="base_link" prefix="right_1" offset_x=" 0.00000" offset_y="-${base_size_y / 2}" offset_z="${wheel_offset_z_from_base_link-0.005}" reflect="1" radius="${wheel_radius_big}" height="${wheel_size_y}" mass="${wheel_mass}"/>
+        <tracked_wheel3 parent="base_link" prefix="right_2" offset_x="-0.25100" offset_y="-${base_size_y / 2}" offset_z="${wheel_offset_z_from_base_link}      " reflect="1" radius="${wheel_radius_big}" height="${wheel_size_y}" mass="${wheel_mass}"/>
         <!--
         <tracked_wheel parent="base_link" prefix="right_3" offset_x="-0.10550" offset_y="-${base_size_y / 2}" offset_z="${wheel_offset_z_from_base_link}      " reflect="1" radius="${wheel_radius_big}" height="${wheel_size_y}" mass="${wheel_mass}"/>
@@ -79,5 +80,4 @@
          -->
         <gazebo>
-        <!-- TODO: make custom plugin for this that doesn't require an imu -->
         <plugin name="diffdrive_plugin_multiwheel" filename="libdiffdrive_plugin_multi_wheel.so">
                 <alwaysOn>true</alwaysOn>
@@ -97,4 +97,29 @@
                 <odometryFrame>odom</odometryFrame>
         </plugin>
+        <!--
+        <plugin name="gazebo_ros_control" filename="libgazebo_ros_control.so">
+            <robotNamespace>/</robotNamespace>
+            <legacyModeNS>true</legacyModeNS>
+        </plugin>
+  <plugin name="skid_steer_drive_controller" filename="libgazebo_ros_skid_steer_drive.so">
+    <updateRate>100.0</updateRate>
+    <robotNamespace>/</robotNamespace>
+    <leftFrontJoint>left_0_wheel_joint</leftFrontJoint>
+    <rightFrontJoint>right_0_wheel_joint</rightFrontJoint>
+    <leftRearJoint>left_2_wheel_joint</leftRearJoint>
+    <rightRearJoint>right_2_wheel_joint</rightRearJoint>
+    <wheelSeparation>0.602</wheelSeparation>
+    <wheelDiameter>0.17</wheelDiameter>
+    <robotBaseFrame>base_link</robotBaseFrame>
+    <MaxForce>5.0</MaxForce>
+    <torque>200</torque>
+    <commandTopic>cmd_vel</commandTopic>
+    <odometryTopic>odom</odometryTopic>
+    <odometryFrame>odom</odometryFrame>
+    <broadcastTF>1</broadcastTF>
+    <covariance_x>0.0</covariance_x>
+    <covariance_y>0.0</covariance_y>
+    <covariance_yaw>0.0</covariance_yaw>
+  </plugin>
         <plugin name="p3d_base_controller" filename="libgazebo_ros_p3d.so">
           <alwaysOn>true</alwaysOn>
@@ -108,8 +133,9 @@
         </plugin>
         <plugin name="imu_controller" filename="libhector_gazebo_ros_imu.so">
+          <robotNamespace>/</robotNamespace>
           <alwaysOn>true</alwaysOn>
           <updateRate>50.0</updateRate>
           <bodyName>base_link</bodyName>
-          <topicName>/gvrbot/imu_quat</topicName>
+          <topicName>/gvrbot/data</topicName>
           <accelDrift>0.0 0.0 0.0</accelDrift>
           <accelGaussianNoise>0.1 0.1 0.1</accelGaussianNoise>
@@ -121,4 +147,5 @@
           <rpyOffset>0 0 0</rpyOffset>
         </plugin>
+-->
         </gazebo>
     </xacro:macro>

Commit message: creating Jackal parallel control and sim for gvrbot

File: models/robots/gvrbot_base.urdf.xacro (robot description, xacro)
@@ -18,7 +18,5 @@
     <xacro:property name="wheel_mass" value="0.1" />
     <xacro:property name="wheel_offset_z_from_base_link" value="-${wheel_radius_big}" />
-      <material name="army_green">
-    <color rgba="${42/255} ${46/255} ${18/255} 1.0"/>
-  </material>
+      <material name="army_green"><color rgba="${42/255} ${46/255} ${18/255} 1.0"/></material>
     <xacro:macro name="gvr_base_macro">
         <!-- Links and Joints (i.e., the robot) -->
