Commit message: wheels turn and ros_control seems to work like with jackal

File: models/robots/model.urdf (robot description, URDF)
Before this commit: robot gvrbot, 12 links, 11 joints
Links:
- removed link chasis_link
- removed link left_0_wheel_link
- removed link left_1_wheel_link
- removed link left_2_wheel_link
- removed link right_0_wheel_link
- removed link right_1_wheel_link
- removed link right_2_wheel_link
- added link chassis_link, mass 25.0; collision box size=0.38 0.3 0.085; visual mesh filename=package://gvrbot/models/meshes/gvrbot_base.STL
- added link front_left_wheel_link, mass 0.477; collision cylinder length=0.04 radius=0.098; visual mesh filename=package://jackal_description/meshes/jackal-wheel.stl
- added link front_right_wheel_link, mass 0.477; collision cylinder length=0.04 radius=0.098; visual mesh filename=package://jackal_description/meshes/jackal-wheel.stl
- added link rear_left_wheel_link, mass 0.477; collision cylinder length=0.04 radius=0.098; visual mesh filename=package://jackal_description/meshes/jackal-wheel.stl
- added link rear_right_wheel_link, mass 0.477; collision cylinder length=0.04 radius=0.098; visual mesh filename=package://jackal_description/meshes/jackal-wheel.stl
Joints:
- removed joint chasis_to_bl
- removed joint left_0_wheel_joint
- removed joint left_1_wheel_joint
- removed joint left_2_wheel_joint
- removed joint right_0_wheel_joint
- removed joint right_1_wheel_joint
- removed joint right_2_wheel_joint
- added joint base_link_joint: type fixed, parent base_link, child chassis_link, origin xyz=0 0 0 rpy=0 0 0
- added joint front_left_wheel: type continuous, parent chassis_link, child front_left_wheel_link, origin xyz=0.22 0.165 -0.07 rpy=0 0 0, axis 0 1 0
- added joint front_right_wheel: type continuous, parent chassis_link, child front_right_wheel_link, origin xyz=0.22 -0.165 -0.07 rpy=0 0 0, axis 0 1 0
- added joint rear_left_wheel: type continuous, parent chassis_link, child rear_left_wheel_link, origin xyz=-0.28 0.165 -0.07 rpy=0 0 0, axis 0 1 0
- added joint rear_right_wheel: type continuous, parent chassis_link, child rear_right_wheel_link, origin xyz=-0.28 -0.165 -0.07 rpy=0 0 0, axis 0 1 0
