Commit message: fixed error in xacro wheel

File: models/robots/single_wheel.urdf.xacro (robot description, xacro)
@@ -1,5 +1,4 @@
 <?xml version="1.0"?>
 <robot xmlns:xacro="http://www.ros.org/wiki/xacro">
-    <xacro:include filename="$(find gvrbot)/models/robots/inertial_tensors.urdf.xacro" />
     <xacro:macro name="wheel" params="prefix *joint_pose">
         <link name="${prefix}_wheel_link">
@@ -17,4 +16,5 @@
         </link>
         <gazebo reference="${prefix}_wheel_link">
+      <material>Gazebo/DarkGrey</material>
         </gazebo>
         <joint name="${prefix}_wheel" type="continuous">
