Commit message: added old changes with old model of gvrbot

File: models/robots/frame_8020.urdf.xacro (robot description, xacro)
@@ -1,3 +1,8 @@
 <robot xmlns:xacro="http://www.ros.org/wiki/xacro">
+    <xacro:include filename="$(find gvrbot)/models/robots/inertial_tensors.urdf.xacro" />
+    <xacro:property name="frame_size_x" value="0.680" />
+    <xacro:property name="frame_size_y" value="0.20" />
+    <xacro:property name="frame_size_z" value="0.30" />
+    <xacro:property name="frame_mass" value="2.89" />
     <xacro:property name="M_PI" value="3.14159"/>
     <xacro:macro name="frame_8020" params="parent offset_x offset_y offset_z">
@@ -9,9 +14,7 @@
         <link name="frame8020_link">
             <inertial>
-              <origin xyz="0.13868 -0.31707 0.28419" rpy="0 0 0" />
-              <mass value="4.2785" />
-              <inertia
-                ixx="0.11494" ixy="-6.8249E-05" ixz="-0.00030429"
-                iyy="0.12359" iyz="-0.001274" izz="0.071887" />
+              <origin xyz="0.0 -0.0 0.0" rpy="0 0 0" />
+              <mass value="${frame_mass}" />
+              <rectangular_prism_tensor mass="${frame_mass}" len_x="${frame_size_x}" len_y="${frame_size_y}" len_z="${frame_size_z}" />
             </inertial>
             <visual>

File: models/robots/gvrbot.urdf.xacro (robot description, xacro)
@@ -1,7 +1,8 @@
 <?xml version="1.0"?>
 <robot name="gvrbot" xmlns:xacro="http://www.ros.org/wiki/xacro">
-    <!-- Included URDF Files    -->
+    <!-- Included URDF Files -->
     <xacro:include filename="$(find gvrbot)/models/robots/gvrbot_base.urdf.xacro" />
     <gvr_base_macro />
+    <!--
     <xacro:include filename="$(find gvrbot)/models/robots/frame_8020.urdf.xacro" />
     <frame_8020 parent="base_link" offset_x="0.28" offset_y="0.135" offset_z="-0.115"/>
@@ -12,3 +13,11 @@
         <origin xyz="-0.028 -0.006 0.46" rpy="0 0 0" />
     </HDL-32E>
+  <xacro:include filename="$(find lms1xx)/urdf/sick_lms1xx.urdf.xacro" />
+    <sick_lms1xx frame="front_laser" topic="/front/scan" />
+    <joint name="front_laser_joint" type="fixed">
+        <origin xyz="-0.028 -0.006 0.56" rpy="0 0 0" />
+      <parent link="base_link" />
+      <child link="front_laser" />
+    </joint>
+      -->
 </robot>

File: models/robots/gvrbot_base.urdf.xacro (robot description, xacro)
@@ -7,8 +7,8 @@
     <!-- Properties (Constants) -->
     <xacro:property name="PI" value="3.1415926535897931" />
-    <xacro:property name="base_size_x" value="0.380" />
-    <xacro:property name="base_size_y" value="0.3" />
-    <xacro:property name="base_size_z" value="0.085" />
-    <xacro:property name="base_mass" value="25.0" />
+    <xacro:property name="base_size_x" value="0.680" />
+    <xacro:property name="base_size_y" value="0.42" />
+    <xacro:property name="base_size_z" value="0.178" />
+    <xacro:property name="base_mass" value="10.89" />
     <xacro:property name="wheel_radius_big" value="0.085" />
     <xacro:property name="wheel_size_y" value="0.0825" />
@@ -17,5 +17,5 @@
     <material name="army_green"><color rgba="${42/255} ${46/255} ${18/255} 1.0"/></material>
     <xacro:macro name="gvr_base_macro">
-        <!-- Links and Joints (i.e., the robot) -->
+        <!-- Links and Joints (i.e., the robot)
         <link name="base_footprint"/>
         <joint name="bf_to_bl" type="fixed">
@@ -24,4 +24,5 @@
           <child link="base_footprint"/>
         </joint>
+        -->
         <link name="base_link"></link>
         <joint name="base_link_joint" type="fixed">
@@ -30,13 +31,19 @@
             <child link="chassis_link" />
         </joint>
+        <link name="imu_link"/>
+        <joint name="imu_to_bl" type="fixed">
+          <origin xyz="0.0 0.0 0.0" rpy="0.0 0.0 0.0" />
+          <parent link="base_link"/>
+          <child link="imu_link"/>
+        </joint>
         <link name="chassis_link">
             <inertial>
                 <mass value="${base_mass}" />
-                <origin xyz="0.0 0.0 0.0" rpy="0 0 0" />
-                <rectangular_prism_tensor mass="${base_mass}" len_x="${base_size_x}" len_y="${base_size_y}" len_z="${base_size_z}" />
+                <origin xyz="${-base_size_x/2} 0 ${base_size_z/2 + 0.05}" rpy="0 0 0" />
+                <box_inertia x="${base_size_x}" y="${base_size_y}" z="${base_size_z}" mass="${base_mass}" />
             </inertial>
             <!-- compare the two visual pieces until they match up in size then delete the mesh -->
             <visual>
-                <origin xyz="${base_size_x - 0.05} 0.0 -${base_size_z * 2}" rpy="0 0 1.57" />
+                <origin xyz="0 0 0" rpy="0 0 ${PI/2}" />
                 <geometry>
                     <mesh filename="package://gvrbot/models/meshes/gvrbot_base.STL"/>
@@ -52,7 +59,7 @@
             </visual-->
             <collision>
-                <origin xyz="0.0 0.0 -0.085" rpy="0 0 0" />
+                <origin xyz="0 0 0" rpy="0 0 ${PI/2}" />
                 <geometry>
-                    <box size="${base_size_x} ${base_size_y} ${base_size_z}" />
+                    <mesh filename="package://gvrbot/models/meshes/gvrbot_base.STL"/>
                 </geometry>
             </collision>
@@ -61,6 +68,7 @@
         <xacro:property name="track" value="0.33" />
         <xacro:property name="wheel_vertical_offset" value="-0.09" />
-        <xacro:property name="wheel_radius" value="0.15" />  <!--  098   -->
+        <xacro:property name="wheel_radius" value="0.15" />
         <xacro:property name="wheel_width" value="0.040" />
+       <!--
         <xacro:wheel prefix="front_left">
             <origin xyz="${wheelbase/2-0.03} ${track/2} ${wheel_vertical_offset}" rpy="0 0 0" />
@@ -95,5 +103,5 @@
                 <updateRate>50.0</updateRate>
                 <bodyName>base_link</bodyName>
-                <topicName>imu/data</topicName>
+                <topicName>/imu/data</topicName>
                 <accelDrift>0.005 0.005 0.005</accelDrift>
                 <accelGaussianNoise>0.005 0.005 0.005</accelGaussianNoise>
@@ -106,4 +114,5 @@
             </plugin>
         </gazebo>
+                -->
     </xacro:macro>
 </robot>

File: models/robots/inertial_tensors.urdf.xacro (robot description, xacro)
@@ -12,3 +12,17 @@
                izz="${ mass / 2 * radius * radius }" />
   </xacro:macro>
+  <xacro:macro name="box_inertia" params="x y z mass">
+      <inertia ixx="${0.0833333 * mass * (y*y + z*z)}" ixy="0.0" ixz="0.0"
+        iyy="${0.0833333 * mass * (x*x + z*z)}" iyz="0.0"
+        izz="${0.0833333 * mass * (x*x + y*y)}" />
+  </xacro:macro>
+  <xacro:macro name="cylinder_inertial" params="radius length mass">
+    <inertial>
+      <mass value="${mass}" />
+      <origin xyz="0 0 0" />
+      <inertia ixx="${0.0833333 * mass * (3 * radius * radius + length * length)}" ixy="0.0" ixz="0.0"
+        iyy="${0.0833333 * mass * (3 * radius * radius + length * length)}" iyz="0.0"
+        izz="${0.5 * mass * radius * radius}" />
+    </inertial>
+  </xacro:macro>
 </robot>
