Commit message: some cleanup but diff drive still not working

File: models/robots/gvrbotJ_base.urdf.xacro (robot description, xacro)
@@ -10,5 +10,5 @@
     <xacro:property name="base_size_y" value="0.42" />
     <xacro:property name="base_size_z" value="0.175" />
-    <xacro:property name="base_mass" value="1.89" />
+    <xacro:property name="base_mass" value="10.89" />
     <xacro:property name="wheel_size_y" value="0.0825" />
     <xacro:property name="wheel_mass" value="0.1" />
@@ -72,4 +72,20 @@
         </xacro:wheel>
         <gazebo>
+            <gazebo>
+              <plugin name="skid_steer_drive_controller" filename="libgazebo_ros_skid_steer_drive.so">
+                <updateRate>100.0</updateRate>
+                <robotNamespace>/</robotNamespace>
+                <leftFrontJoint>front_left_wheel_joint</leftFrontJoint>
+                <rightFrontJoint>front_right_wheel_joint</rightFrontJoint>
+                <leftRearJoint>back_left_wheel_joint</leftRearJoint>
+                <rightRearJoint>back_right_wheel_joint</rightRearJoint>
+                <wheelSeparation>0.4</wheelSeparation>
+                <wheelDiameter>0.215</wheelDiameter>
+                <robotBaseFrame>base_link</robotBaseFrame>
+                <torque>20</torque>
+                <topicName>cmd_vel</topicName>
+                <broadcastTF>false</broadcastTF>
+              </plugin>
+            </gazebo>
             <plugin name="gazebo_ros_control" filename="libgazebo_ros_control.so">
                 <robotNamespace>/</robotNamespace>

File: models/robots/single_wheel.urdf.xacro (robot description, xacro)
@@ -2,4 +2,6 @@
 <robot xmlns:xacro="http://www.ros.org/wiki/xacro">
     <xacro:macro name="wheel" params="prefix *joint_pose">
+        <xacro:property name="wheel_radius" value="0.14" />
+        <xacro:property name="wheel_width" value="0.040" />
         <link name="${prefix}_wheel_link">
             <collision>
@@ -16,5 +18,11 @@
         </link>
         <gazebo reference="${prefix}_wheel_link">
-      <material>Gazebo/DarkGrey</material>
+              <material>Gazebo/DarkGrey</material>
+              <selfCollide>false</selfCollide>
+              <mu1 value="0.5"/>
+              <mu2 value="0.5"/>
+              <kp value="10000000.0" />
+              <kd value="1" />
+              <fdir1 value="1 0 0"/>
         </gazebo>
         <joint name="${prefix}_wheel" type="continuous">
