Commit message: added 8020 frame and moved compass

File: models/urdf/frame_8020.urdf.xacro (robot description, xacro)
@@ -1,12 +1,12 @@
 <robot xmlns:xacro="http://www.ros.org/wiki/xacro">
     <xacro:include filename="$(find gvrbot)/models/urdf/inertial_tensors.urdf.xacro" />
-    <xacro:property name="frame_size_x" value="0.680" />
-    <xacro:property name="frame_size_y" value="0.20" />
-    <xacro:property name="frame_size_z" value="0.30" />
+    <xacro:property name="frame_length" value="0.680" />
+    <xacro:property name="frame_width" value="0.20" />
+    <xacro:property name="frame_height" value="0.30" />
     <xacro:property name="frame_mass" value="2.89" />
     <xacro:property name="M_PI" value="3.14159"/>
     <xacro:macro name="frame_8020" params="parent offset_x offset_y offset_z">
         <joint name="frame_8020_joint" type="fixed">
-            <origin xyz="${offset_x} ${offset_y} ${offset_z}" rpy="0 0 ${-M_PI/2}" />
+            <origin xyz="${offset_x} ${offset_y} ${offset_z}" rpy="0 0 ${PI/2}" />
             <parent link="${parent}" />
             <child link="frame8020_link" />
@@ -14,7 +14,7 @@
         <link name="frame8020_link">
             <inertial>
-              <origin xyz="0.0 -0.0 0.0" rpy="0 0 0" />
+              <origin xyz="0.135 -0.315 0.2" rpy="${PI/2} 0 ${PI/2}" />
               <mass value="${frame_mass}" />
-              <rectangular_prism_tensor mass="${frame_mass}" len_x="${frame_size_x}" len_y="${frame_size_y}" len_z="${frame_size_z}" />
+                <box_inertia x="${frame_length}" y="${frame_width}" z="${frame_height}" mass="${frame_mass}" />
             </inertial>
             <visual>

File: models/urdf/gvrbot2.urdf.xacro (robot description, xacro)
@@ -1,4 +1,5 @@
 <?xml version="1.0"?>
 <robot name="gvrbot" xmlns:xacro="http://www.ros.org/wiki/xacro">
+    <xacro:include filename="$(find gvrbot)/models/urdf/inertial_tensors.urdf.xacro" />
   <xacro:property name="PI" value="3.1415926535897931" />
   <xacro:property name="wheelbase" value="0.262" />
@@ -8,7 +9,8 @@
   <xacro:property name="wheel_radius" value="0.098" />
   <xacro:property name="wheel_width" value="0.040" />
-  <xacro:property name="chassis_length" value="0.420" />
-  <xacro:property name="chassis_width" value="0.310" />
-  <xacro:property name="chassis_height" value="0.184" />
+  <xacro:property name="chassis_length" value="0.680" />
+  <xacro:property name="chassis_width" value="0.42" />
+  <xacro:property name="chassis_height" value="0.178" />
+  <xacro:property name="chassis_mass" value="10.89" />
   <xacro:property name="dummy_inertia" value="1e-09"/>
   <xacro:property name="mount_spacing" value="0.120" />
@@ -106,12 +108,9 @@
     <inertial>
       <!-- Center of mass -->
-      <origin xyz="0.012  0.002 0.067" rpy="0 0 0"/>
-      <mass value="16.523"/>
+        <origin xyz="-0.005 0 0.03" rpy="0 0 0" />
+        <mass value="${chassis_mass}"/>
       <!-- Moments of inertia: ( chassis without wheels ) -->
-      <inertia
-        ixx="0.3136" ixy="-0.0008" ixz="0.0164"
-        iyy="0.3922" iyz="-0.0009"
-        izz="0.4485"/>
-      </inertial>
+      <box_inertia x="${chassis_length}" y="${chassis_width}" z="${chassis_height}" mass="${chassis_mass}" />
+    </inertial>
   </link>
   <!-- TODO: Make this internal_imu_link or something, and use a mixed-in xacro
@@ -136,5 +135,5 @@
         <cylinder radius="0.026" length="0.016" />
       </geometry>
-      <origin xyz="0 0 0.008" />
+      <origin xyz="0.08 -0.03 0.235" />
       <material name="black" />
     </visual>
@@ -165,3 +164,6 @@
   <!-- Bring in simulation data for Gazebo. -->
   <xacro:include filename="$(find gvrbot)/models/urdf/gvrbot.gazebo" />
+  <!-- Add 8020 Frame. -->
+    <xacro:include filename="$(find gvrbot)/models/urdf/frame_8020.urdf.xacro" />
+    <frame_8020 parent="base_link" offset_x="-0.315" offset_y="-0.1389" offset_z="-0.01"/>
 </robot>
