Commit message: inertia fxd, with 2d lidar, gps, and IMU working

File: models/urdf/frame_8020.urdfv2.xacro (robot description, xacro)
@@ -8,5 +8,6 @@
     <xacro:macro name="frame_8020" params="parent offset_x offset_y offset_z">
         <joint name="frame_8020_joint" type="fixed">
-            <origin xyz="${offset_x} ${offset_y} ${offset_z}" rpy="0 0 0" />
+            <!-- <origin xyz="${offset_x} ${offset_y} ${offset_z}" rpy="0 0 ${PI/2}" />   -->
+          <origin xyz="0 0 0" rpy="0 0 0" />
             <parent link="${parent}" />
             <child link="frame8020_link" />
@@ -14,7 +15,8 @@
         <link name="frame8020_link">
             <inertial>
+              <!-- <origin xyz="0.135 -0.315 0.2" rpy="${PI/2} 0 ${PI/2}" /> -->
               <origin xyz="0.331 0.117 0.077" rpy="0 0 0" />
               <mass value="${frame_mass}" />
-                <xacro:box_inertia x="${frame_length}" y="${frame_width}" z="${frame_height}" mass="${frame_mass}" />
+                <box_inertia x="${frame_length}" y="${frame_width}" z="${frame_height}" mass="${frame_mass}" />
             </inertial>
             <visual>

File: models/urdf/gvrbot.urdf.xacro (robot description, xacro)
@@ -90,5 +90,4 @@
         <box size="0.01 0.01 0.01"/>
       </geometry>
-    <script>Gazebo/Orange</script>
     </visual>
   </link>
@@ -120,9 +119,5 @@
     </inertial>
   </link>
-  <!-- TODO: Make this internal_imu_link or something, and use a mixed-in xacro
-       to supply the joint between it and imu_link. This is important so that imu_link
-       always points to the "active" IMU. When an upgrade IMU is connected, the
-       internal_imu_link should remain, but imu_link should point to the upgrade one. -->
-  <link name="imu_link">
+ <link name="imu_link">
     <inertial>
       <mass value="0.001"/>
@@ -157,9 +152,7 @@
   </joint>
       <xacro:include filename="$(find gvrbot)/models/urdf/hokuyo_ust10.urdf.xacro" />
-      <xacro:hokuyo_ust10_mount prefix="top"
-                          topic="front/scan"/>
+      <xacro:hokuyo_ust10_mount prefix="top"  topic="front/scan"/>
       <joint name="top_laser_mount_joint" type="fixed">
-        <origin xyz="0.1 0 0"
-                rpy="0 0 0" />
+        <origin xyz="0.1 0 0" rpy="0 0 0" />
         <parent link="top_mount" />
         <child link="top_laser_mount" />
@@ -167,5 +160,5 @@
   <!-- Bring in simulation data for Gazebo. -->
   <xacro:include filename="$(find gvrbot)/models/urdf/gvrbot.gazebo" />
-  <!-- Add 8020 Frame. -->
+  <!-- Add 8020 Frame.  -->
     <xacro:include filename="$(find gvrbot)/models/urdf/frame_8020.urdf.xacro" />
     <xacro:frame_8020 parent="base_link" offset_x="-0.335" offset_y="-0.117" offset_z="0.132"/>
