Commit message: D200 depth camera working

File: models/urdf/gvrbot.urdf.xacro (robot description, xacro)
@@ -130,19 +130,5 @@
     <child link="imu_link" />
   </joint>
-  <!-- TODO: Same note as applies to imu_link -->
-  <link name="navsat_link">
-    <visual>
-      <geometry>
-        <cylinder radius="0.026" length="0.016" />
-      </geometry>
-      <origin xyz="0 0 0" />
-      <material name="black" />
-    </visual>
-  </link>
-  <joint name="navsat_joint" type="fixed">
-        <parent link="top_mount" />
-    <child link="navsat_link" />
-    <origin xyz="-0.1 0.1 0" />
-  </joint>
+  <!-- Create a mount point in the center of top plate -->
   <link name="top_mount"></link>
   <joint name="top_mount_joint" type="fixed">
@@ -151,4 +137,20 @@
     <origin xyz="-0.004 0 0.406" />
   </joint>
+  <!-- Add GPS to top left of top plate on robot. -->
+  <link name="navsat_link">
+    <visual>
+      <geometry>
+        <cylinder radius="0.026" length="0.016" />
+      </geometry>
+      <origin xyz="0 0 0" />
+      <material name="black" />
+    </visual>
+  </link>
+  <joint name="navsat_joint" type="fixed">
+        <parent link="top_mount" />
+    <child link="navsat_link" />
+    <origin xyz="-0.1 0.1 0" />
+  </joint>
+  <!-- Add Hokuyo UST10 2d Lidar to front of robot. -->
       <xacro:include filename="$(find gvrbot)/models/urdf/hokuyo_ust10.urdf.xacro" />
       <xacro:hokuyo_ust10_mount prefix="top"  topic="front/scan"/>
@@ -160,4 +162,65 @@
   <!-- Bring in simulation data for Gazebo. -->
   <xacro:include filename="$(find gvrbot)/models/urdf/gvrbot.gazebo" />
+  <xacro:property name="r200_cam_rgb_px" value="0.005"/>
+  <xacro:property name="r200_cam_rgb_py" value="0.018"/>
+  <xacro:property name="r200_cam_rgb_pz" value="0.013"/>
+  <xacro:property name="r200_cam_depth_offset" value="0.01"/>
+  <!-- Add Realsense D200 joint to front of robot. -->
+  <joint name="depthcamera_joint" type="fixed">
+        <parent link="top_mount" />
+    <child link="camera_rgb_frame" />
+    <origin xyz="0.14 0 0.014" />
+  </joint>
+  <joint name="camera_joint" type="fixed">
+    <origin xyz="0.064 -0.065 0.094" rpy="0 0 0"/>
+    <parent link="base_link"/>
+    <child link="camera_link"/>
+  </joint>
+  <link name="camera_link">
+    <visual>
+     <origin xyz="0 0 0" rpy="1.57 0 1.57"/>
+      <geometry>
+       <mesh filename="package://turtlebot3_description/meshes/sensors/r200.dae" />
+      </geometry>
+    </visual>
+    <collision>
+      <origin xyz="0.003 0.065 0.007" rpy="0 0 0"/>
+      <geometry>
+        <box size="0.012 0.132 0.020"/>
+      </geometry>
+    </collision>
+    <!-- This inertial field needs doesn't contain reliable data!! -->
+<!--   <inertial>
+      <mass value="0.564" />
+      <origin xyz="0 0 0" />
+      <inertia ixx="0.003881243" ixy="0.0" ixz="0.0"
+               iyy="0.000498940" iyz="0.0"
+               izz="0.003879257" />
+    </inertial>-->
+  </link>
+  <joint name="camera_rgb_joint" type="fixed">
+    <origin xyz="${r200_cam_rgb_px} ${r200_cam_rgb_py} ${r200_cam_rgb_pz}" rpy="0 0 0"/>
+    <parent link="camera_link"/>
+    <child link="camera_rgb_frame"/>
+  </joint>
+  <link name="camera_rgb_frame"/>
+  <joint name="camera_rgb_optical_joint" type="fixed">
+    <origin xyz="0 0 0" rpy="-1.57 0 -1.57"/>
+    <parent link="camera_rgb_frame"/>
+    <child link="camera_rgb_optical_frame"/>
+  </joint>
+  <link name="camera_rgb_optical_frame"/>
+  <joint name="camera_depth_joint" type="fixed">
+    <origin xyz="${r200_cam_rgb_px} ${r200_cam_rgb_py + r200_cam_depth_offset} ${r200_cam_rgb_pz}" rpy="0 0 0"/>
+    <parent link="camera_link"/>
+    <child link="camera_depth_frame"/>
+  </joint>
+  <link name="camera_depth_frame"/>
+  <joint name="camera_depth_optical_joint" type="fixed">
+    <origin xyz="0 0 0" rpy="-1.57 0 -1.57"/>
+    <parent link="camera_depth_frame"/>
+    <child link="camera_depth_optical_frame"/>
+  </joint>
+  <link name="camera_depth_optical_frame"/>
   <!-- Add 8020 Frame.  -->
     <xacro:include filename="$(find gvrbot)/models/urdf/frame_8020.urdf.xacro" />

File: models/urdf/hokuyo_ust10.urdf.xacro (robot description, xacro)
@@ -13,5 +13,5 @@
       </link>
       <gazebo reference="${frame}">
-        <turnGravityOff>true</turnGravityOff>
+        <turnGravityOff>false</turnGravityOff>
         <sensor type="ray" name="${frame}">
           <pose>0 0 0 0 0 0</pose>

Commit message: working depth camera with D435 being shown

File: models/urdf/gvrbot.urdf.xacro (robot description, xacro)
@@ -162,67 +162,12 @@
   <!-- Bring in simulation data for Gazebo. -->
   <xacro:include filename="$(find gvrbot)/models/urdf/gvrbot.gazebo" />
-  <xacro:property name="r200_cam_rgb_px" value="0.005"/>
-  <xacro:property name="r200_cam_rgb_py" value="0.018"/>
-  <xacro:property name="r200_cam_rgb_pz" value="0.013"/>
-  <xacro:property name="r200_cam_depth_offset" value="0.01"/>
-  <!-- Add Realsense D200 joint to front of robot. -->
-  <joint name="depthcamera_joint" type="fixed">
-        <parent link="top_mount" />
-    <child link="camera_rgb_frame" />
-    <origin xyz="0.14 0 0.014" />
-  </joint>
-  <joint name="camera_joint" type="fixed">
-    <origin xyz="0.064 -0.065 0.094" rpy="0 0 0"/>
-    <parent link="base_link"/>
-    <child link="camera_link"/>
-  </joint>
-  <link name="camera_link">
-    <visual>
-     <origin xyz="0 0 0" rpy="1.57 0 1.57"/>
-      <geometry>
-       <mesh filename="package://turtlebot3_description/meshes/sensors/r200.dae" />
-      </geometry>
-    </visual>
-    <collision>
-      <origin xyz="0.003 0.065 0.007" rpy="0 0 0"/>
-      <geometry>
-        <box size="0.012 0.132 0.020"/>
-      </geometry>
-    </collision>
-    <!-- This inertial field needs doesn't contain reliable data!! -->
-<!--   <inertial>
-      <mass value="0.564" />
-      <origin xyz="0 0 0" />
-      <inertia ixx="0.003881243" ixy="0.0" ixz="0.0"
-               iyy="0.000498940" iyz="0.0"
-               izz="0.003879257" />
-    </inertial>-->
-  </link>
-  <joint name="camera_rgb_joint" type="fixed">
-    <origin xyz="${r200_cam_rgb_px} ${r200_cam_rgb_py} ${r200_cam_rgb_pz}" rpy="0 0 0"/>
-    <parent link="camera_link"/>
-    <child link="camera_rgb_frame"/>
-  </joint>
-  <link name="camera_rgb_frame"/>
-  <joint name="camera_rgb_optical_joint" type="fixed">
-    <origin xyz="0 0 0" rpy="-1.57 0 -1.57"/>
-    <parent link="camera_rgb_frame"/>
-    <child link="camera_rgb_optical_frame"/>
-  </joint>
-  <link name="camera_rgb_optical_frame"/>
-  <joint name="camera_depth_joint" type="fixed">
-    <origin xyz="${r200_cam_rgb_px} ${r200_cam_rgb_py + r200_cam_depth_offset} ${r200_cam_rgb_pz}" rpy="0 0 0"/>
-    <parent link="camera_link"/>
-    <child link="camera_depth_frame"/>
-  </joint>
-  <link name="camera_depth_frame"/>
-  <joint name="camera_depth_optical_joint" type="fixed">
-    <origin xyz="0 0 0" rpy="-1.57 0 -1.57"/>
-    <parent link="camera_depth_frame"/>
-    <child link="camera_depth_optical_frame"/>
-  </joint>
-  <link name="camera_depth_optical_frame"/>
   <!-- Add 8020 Frame.  -->
     <xacro:include filename="$(find gvrbot)/models/urdf/frame_8020.urdf.xacro" />
     <xacro:frame_8020 parent="base_link" offset_x="-0.335" offset_y="-0.117" offset_z="0.132"/>
+  <!-- Add D435 Depth Sensor.  -->
+    <xacro:arg name="use_nominal_extrinsics" default="false"/>
+  <xacro:include filename="$(find gvrbot)/models/urdf/_d435.urdf.xacro" />
+  <xacro:sensor_d435 parent="top_mount" use_nominal_extrinsics="$(arg use_nominal_extrinsics)">
+    <origin xyz="0.14 0 -0.04" rpy="0 0 0"/>
+  </xacro:sensor_d435>
 </robot>
