Commit message: fixed inertia for realsense camera

File: models/urdf/_d435.urdf.xacro (robot description, xacro)
@@ -8,4 +8,5 @@
 <robot name="sensor_d435" xmlns:xacro="http://ros.org/wiki/xacro">
   <!-- Includes -->
+    <xacro:include filename="$(find gvrbot)/models/urdf/inertial_tensors.urdf.xacro" />
   <xacro:include filename="$(find realsense2_description)/urdf/_materials.urdf.xacro" />
   <xacro:macro name="sensor_d435" params="parent *origin name:=camera use_nominal_extrinsics:=false">
@@ -63,7 +64,7 @@
       <inertial>
         <!-- The following are not reliable values, and should not be used for modeling -->
-        <mass value="0.564" />
+        <mass value="0.072" />
         <origin xyz="0 0 0" />
-        <inertia ixx="0.003881243" ixy="0.0" ixz="0.0" iyy="0.000498940" iyz="0.0" izz="0.003879257" />
+      <xacro:box_inertia x="0.09" y="0.025" z="0.025" mass="${chassis_mass}" />
       </inertial>
     </link>

File: models/urdf/gvrbot.urdf.xacro (robot description, xacro)
@@ -165,5 +165,5 @@
     <xacro:include filename="$(find gvrbot)/models/urdf/frame_8020.urdf.xacro" />
     <xacro:frame_8020 parent="base_link" offset_x="-0.335" offset_y="-0.117" offset_z="0.132"/>
-  <!-- Add D435 Depth Sensor.  -->
+  <!-- Add D435 Depth Sensor.   -->
     <xacro:arg name="use_nominal_extrinsics" default="true"/>
   <xacro:include filename="$(find gvrbot)/models/urdf/_d435.urdf.xacro" />
